Commit message: add params in xacro

File: car_sim/fwd_description/urdf/imu.xacro (robot description, xacro)
@@ -1,5 +1,5 @@
 <?xml version="1.0"?>
 <robot name="RMP_1" xmlns:xacro="http://www.ros.org/wiki/xacro" >
-    <xacro:macro name="imu" params="prefix">
+    <xacro:macro name="imu" params="prefix robot_name">
         <link name="${prefix}_link">
             <inertial>
@@ -31,15 +31,15 @@
             <sensor name="imu_sensor" type="imu">
                 <always_on>true</always_on>
-                <update_rate>100</update_rate>
+                <update_rate>10</update_rate>
                 <visualize>true</visualize>
-                <topic>/imu</topic>
+                <topic>imu</topic>
                 <plugin filename="libgazebo_ros_imu_sensor.so" name="imu_plugin">
-                    <topicName>/imu</topicName>
+                    <topicName>imu</topicName>
                     <bodyName>imu_link</bodyName>
-                    <updateRateHZ>0.0</updateRateHZ>
+                    <updateRateHZ>10.0</updateRateHZ>
                     <gaussianNoise>0.0</gaussianNoise>
                     <xyzOffset>0 0 0</xyzOffset>
                     <rpyOffset>0 0 0</rpyOffset>
-                    <frameName>imu_link</frameName>
+                    <frameName>${robot_name}/imu_link</frameName>
                 </plugin>
                 <!--pose>0 0 0 0 0 0</pose-->

File: car_sim/fwd_description/urdf/mini_4wd/mini4wd_camera.xacro (robot description, xacro)
@@ -2,5 +2,5 @@
 <robot name="RMP_1" xmlns:xacro="http://www.ros.org/wiki/xacro">
     <!-- macro define astra_camera-->
-    <xacro:macro name="astra_camera" params="prefix">
+    <xacro:macro name="astra_camera" params="prefix robot_name">
     <!--Defining camera_link -->
     <link name="${prefix}_link">
@@ -62,5 +62,5 @@
                     <cameraInfoTopicName>rgb/camera_info</cameraInfoTopicName>
                     <depthImageCameraInfoTopicName>depth/camera_info</depthImageCameraInfoTopicName>
-                    <frameName>${prefix}_frame_optical</frameName>
+                    <frameName>${robot_name}/${prefix}_frame_optical</frameName>
                     <baseline>0.1</baseline>
                     <distortion_k1>0.0</distortion_k1>

File: car_sim/fwd_description/urdf/mini_4wd/mini4wd_rplidar.xacro (robot description, xacro)
@@ -1,5 +1,5 @@
 <?xml version="1.0"?>
 <robot name="RMP_1" xmlns:xacro="http://www.ros.org/wiki/xacro">
-    <xacro:macro name="rplidar" params="LA">
+    <xacro:macro name="rplidar" params="LA robot_name">
         <!-- define rplidar_link -->
         <link name="${LA}_link">
@@ -49,5 +49,5 @@
                 <plugin name="gazebo_rplidar" filename="libgazebo_ros_laser.so">
                     <topicName>scan</topicName>
-                    <frameName>laser_link</frameName>
+                    <frameName>${robot_name}/laser_link</frameName>
                 </plugin>
             </sensor>

File: car_sim/fwd_description/urdf/mini_4wd/mini_4wd.xacro (robot description, xacro)
@@ -2,4 +2,5 @@
 <robot name="RMP_1" xmlns:xacro="http://www.ros.org/wiki/xacro">
     <!--M_PI-->
+    <xacro:arg name="robot_name" default="RMP_2"/>
     <xacro:property name="M_PI" value="3.1415926535897931" />
     <!--rplidar description-->
@@ -63,6 +64,6 @@
       <child link="imu_link"/>
     </joint>
-    <xacro:imu prefix="imu"/>
-    <xacro:astra_camera prefix="camera"/>
+    <xacro:imu prefix="imu" robot_name="$(arg robot_name)"/>
+    <xacro:astra_camera prefix="camera" robot_name="$(arg robot_name)"/>
     <xacro:joint_choose LR="right" FR="front" >
         <origin xyz="${front_wheel_position_x} ${right_wheel_position_y} ${wheel_position_z} " rpy="0 0 0"/>
@@ -125,4 +126,4 @@
     <xacro:transmission_choose LR="right" FR="rear"  />
     <xacro:transmission_choose LR="left"  FR="rear"  />
-    <xacro:rplidar LA="laser"/>
+    <xacro:rplidar LA="laser" robot_name="$(arg robot_name)"/>
 </robot>
